File: PCB_Design/ADC.brd (EAGLE design)
At the start: 44.2 x 44.2 mm, 15 parts, among them J1-0 AD_CH0- GND option, J1-1 AD_CH1- GND option, J1-2 AD_CH2- GND option, J1-3 AD_CH3- GND option, J1-4 AD_CH4- GND option, J1-5 AD_CH5- GND option, J2 Input Screw-terminal Connector, J3 PMOD Interface Connector, X1 4MHz

Commit message: Add files via upload
Parts:
- X1: value 4MHz -> 4MHZ; device SparkFun-Clocks:CRYSTAL-SMD-MC-146 -> CalPlug:HC-49S
- moved X1 7.17 mm to (23.2, 9.40), turned to 0 degrees
- moved C1 1.02 mm to (17.5, 14.0)
- moved C2 1.02 mm to (24.9, 14.0)
Connections:
- new net N$1: C2.2
- net GND: no longer C2.2
- net OSC_1: now also X1.1; no longer X1.P$1
- net OSC_2: now also X1.2; no longer X1.P$2
Routing:
- net OSC_2: track 8.15 -> 19.4 mm
- net ADC_DR_A: track 43.9 -> 51.9 mm
- net ADC_DR_B: track 43.3 -> 51.2 mm
- net ADC_DR_C: track 43.3 -> 50.8 mm
- net OSC_1: track 8.13 -> 15.1 mm
